File: QL_diren_keyboard_adapter.kicad_sch (KiCad schematic)
At the start: 12 parts, among them J1 Conn_01x20_Pin, J2 Conn_01x20_Pin, J3 Conn_01x05, J4 Conn_01x02, J5 Conn_01x03, U1 8749, U2 PIC16C5X, Y1 20Mhz

Commit message: updated
Parts:
- C1, C2: value 27p -> 15p
- J1, J2: value Conn_01x20_Pin -> Turned Pins 1x20
- J4: value Conn_01x02 -> JUMPER PINS x02
- J5: value Conn_01x03 -> JUMPER PINS x03
- U1: value 8749 -> SOCKET 40 PIN
- U2: value PIC16C5X -> PIC16C57-HS/SO; footprint Package_SO:SOP-28_8.4x18.16mm_P1.27mm -> Package_SO:SOIC-28W_7.5x17.9mm_P1.27mm; symbol MCU_Microchip_PIC16:PIC16F84-XXP -> 8bits:PIC16C5X-xx/SO
- Y1: value 20Mhz -> 10Mhz
Connections:
- net +5V: now also U2.1 (TOCKI), U2.2 (VDD); no longer U2.3 (VDD), U2.4 (VDD)
- net GND: now also U2.4 (VSS); no longer U2.1 (VSS), U2.5 (RA0)
- no-connect marks 1 -> 0
Other:
- moved on the sheet: C1
